Commit message: old stuff in urdf

File: urdf/simple_pan_tilt.urdf (robot description, URDF)
Before this commit: robot simple_pan_tilt, 3 links, 2 joints
Links:
- link pan_link: geometry collision cylinder length=0.4 radius=0.06; visual cylinder length=0.4 radius=0.06
Joints:
- joint tilt_joint: origin xyz=0 0 0.2 -> xyz=0 0 0.3
